File: Eagle Files/8x LED Trieber Stage_01.sch (EAGLE design)
At the start: 98 parts, among them IC10 CAT4101, IC11 CAT4101, IC12 CAT4101, IC13 CAT4101, IC2 7805TV, IC3 ATmega168 (LICHT), IC4 CAT4101, IC6 74LS14D, IC7 CAT4101, IC8 CAT4101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

Commit message: Arduino and Eagle Fixes
Channels in Arduino Coded fixed, Annotations in eagle added
Other:
- note added: "8 Fach LED Driver 10W Stage Edition - TLC5940, Atmega, - 8-channel LED driver - Midi In and Through moritz@sonicrobots.com"
- note removed: "8 Fach LED Treiber 10W Stage Edition - TLC5940, Atmega, - 8-Fach LED Treiber - Midi In and Through"
Changed lines of the file:
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@@
 <plain>
 <text x="149.86" y="124.46" size="1.778" layer="91"></text>
-<text x="360.68" y="363.22" size="5.08" layer="91">8 Fach LED Treiber 10W Stage Edition
+<text x="360.68" y="363.22" size="5.08" layer="91">8 Fach LED Driver 10W Stage Edition
 - TLC5940, Atmega,
-- 8-Fach LED Treiber
+- 8-channel LED driver
 - Midi In and Through
-</text>
+moritz@sonicrobots.com</text>
 <text x="256.54" y="347.98" size="1.016" layer="91">Arduino Pin 12</text>
 <text x="256.54" y="345.44" size="1.27" layer="91">Arduino Pin 11</text>
